Commit message: all three sensors not crashing

File: rover_description/robots/rover.urdf.xacro (robot description, xacro)
@@ -2,6 +2,6 @@
 <robot name="rover" xmlns:xacro="http://www.ros.org/wiki/xacro">
     <!-- Include macros -->
-    <xacro:include filename="$(find rover_description)/urdf/materials.xacro"/>
-    <xacro:include filename="$(find rover_description)/urdf/inertials.xacro"/>
+    <xacro:include filename="$(find rover_description)/urdf/materials.xacro" />
+    <xacro:include filename="$(find rover_description)/urdf/inertials.xacro" />
     <xacro:include filename="$(find rover_description)/urdf/bases/body.urdf.xacro" />
     <xacro:include filename="$(find rover_description)/urdf/bases/differential.urdf.xacro" />
@@ -13,4 +13,5 @@
     <xacro:include filename="$(find rover_description)/urdf/sensors/all_sensors.urdf.xacro" />
     <!-- Gazebo ROS2 Control -->
+    <!--
     <gazebo>
         <plugin filename="libgazebo_ros2_control.so" name="gazebo_ros2_control">
@@ -139,5 +140,7 @@
         </joint>
     </ros2_control>
-    <!-- The base link -->
+    -->
+   <!-- The base link - the reference link for the entire model -->
+    <link name="base_footprint" /> <!-- dummy link for gazebo -->
     <link name="base_link">
         <visual>
@@ -148,15 +151,28 @@
             <material name="orange" />
         </visual>
+        <collision>
+            <origin rpy="0 0 0" xyz="0 0 0" />
+            <geometry>
+                <box size="0.01 0.01 0.01"/>
+            </geometry>
+        </collision>
+        <xacro:solid_cuboid_inertial
+            rpy="0 0 0" xyz="0 0 0"
+            mass="0.01"
+            x="0.01" y="0.01" z="0.01" />
     </link>
-    <gazebo reference="base_link">
-        <material>Gazebo/Orange</material>
-    </gazebo>
+    <joint name="base_joint" type="fixed">
+        <parent link="base_footprint"/>
+        <origin rpy="0 0 0" xyz="0 0 1.0"/>
+        <child link="base_link"/>
+        <axis xyz="0 0 1"/>
+    </joint>
     <!-- body -->
     <xacro:body parent="base_link" />
     <xacro:differential parent="base_link" />
+    <xacro:rocker parent="base_link" lat_label="left" reflect="1"/>
+    <xacro:rocker parent="base_link" lat_label="right" reflect="-1"/>
     <xacro:turnbuckle lat_label="left" reflect="1"/>
     <xacro:turnbuckle lat_label="right" reflect="-1"/>
-    <xacro:rocker parent="base_link" lat_label="left" reflect="1"/>
-    <xacro:rocker parent="base_link" lat_label="right" reflect="-1"/>
     <xacro:bogie lat_label="left" reflect="1"/>
     <xacro:bogie lat_label="right" reflect="-1"/>
@@ -166,12 +182,11 @@
     </xacro:sensor_hokuyo>
     <xacro:sensor_imu prefix="imu" parent="base_link">
-        <!-- <origin xyz="-0.32 0 0.05" rpy="0 0.5 0"/> -->
         <origin xyz="0 0 -0.04" rpy="0 0 0"/>
     </xacro:sensor_imu>
     <xacro:sensor_asus_xtion prefix="camera" parent="base_link">
         <origin xyz="0.215 0 0.065" rpy="0 0.4 0"/>
-        <!-- <origin xyz="0.212 0 0.065" rpy="0 0 0"/> -->
     </xacro:sensor_asus_xtion>
     <!-- wheels -->
+    <!--
     <xacro:corner_link lon_label="front" lat_label="left" reflect="1"/>
     <xacro:corner_link lon_label="front" lat_label="right" reflect="-1"/>
@@ -194,3 +209,4 @@
     <xacro:corner_wheel_joint lon_label="back" lat_label="left" reflect="1"/>
     <xacro:corner_wheel_joint lon_label="back" lat_label="right" reflect="-1"/>
+    -->
 </robot>

File: rover_description/urdf/bases/body.urdf.xacro (robot description, xacro)
@@ -45,7 +45,4 @@
                 x="${body_box_length}" y="${body_box_width}" z="${body_box_depth}" />
         </link>
-        <gazebo reference="body_box_link">
-            <material>Gazebo/White</material>
-        </gazebo>
         <joint name="body_box_joint" type="fixed">
             <origin rpy="0 0 0" xyz="0 0 0"/>

File: rover_description/urdf/bases/bogie.urdf.xacro (robot description, xacro)
@@ -45,8 +45,15 @@
                 x="${bogie_box_length}" y="${bogie_box_width}" z="${bogie_box_depth}" />
         </link>
-        <gazebo reference="${lat_label}_bogie_link">
-            <material>Gazebo/White</material>
-        </gazebo>
-        <!-- joint -->
+        <!-- Fixed Bogie Joint  (for testing) -->
+        <!--
+        <xacro:macro name="bogie_joint" params="lat_label reflect">
+            <joint name="${lat_label}_bogie_joint" type="fixed">
+                <origin rpy="0 0 0" xyz="-1.181 ${reflect * 0.025} -0.062"/>
+                <parent link="${lat_label}_rocker_link" />
+                <child link="${lat_label}_bogie_link" />
+            </joint>
+        </xacro:macro>
+        -->
+        <!-- Articulated joint -->
         <joint name="${lat_label}_bogie_joint" type="revolute">
             <origin rpy="0 0 0" xyz="-0.181 ${reflect * 0.025} -0.062"/>
@@ -60,8 +67,4 @@
             <child link="${lat_label}_bogie_link" />
         </joint>
-        <gazebo reference="${lat_label}_bogie_joint">
-            <provideFeedback>true</provideFeedback>
-            <implicitSpringDamper>true</implicitSpringDamper>
-        </gazebo>
     </xacro:macro>
 </robot>

File: rover_description/urdf/bases/differential.urdf.xacro (robot description, xacro)
@@ -45,7 +45,4 @@
                 x="${differential_box_length}" y="${differential_box_width}" z="${differential_box_depth}" />
         </link>
-        <gazebo reference="diff_brace_link">
-            <material>Gazebo/White</material>
-        </gazebo>
         <joint name="diff_brace_joint" type="revolute">
             <origin rpy="0 0 0" xyz="0 0 0.0681"/>
@@ -59,8 +56,4 @@
             <child link="diff_brace_link" />
         </joint>
-        <gazebo reference="diff_brace_joint">
-            <provideFeedback>true</provideFeedback>
-            <implicitSpringDamper>true</implicitSpringDamper>
-        </gazebo>
     </xacro:macro>
 </robot>

File: rover_description/urdf/bases/rocker.urdf.xacro (robot description, xacro)
@@ -46,8 +46,13 @@
                 x="${rocker_box_length}" y="${rocker_box_width}" z="${rocker_box_depth}" />
         </link>
-        <gazebo reference="${lat_label}_rocker_link">
-            <material>Gazebo/White</material>
-        </gazebo>
-        <!-- joint -->
+        <!-- Fixed Rocker Joint (for testing)  -->
+        <!--
+            <joint name="${lat_label}_rocker_joint" type="fixed">
+                <origin rpy="0 0 0" xyz="0.071 ${reflect * 0.154} 0.0118"/>
+                <parent link="base_link" />
+                <child link="${lat_label}_rocker_link" />
+            </joint>
+        -->
+        <!-- Articulated joint -->
         <joint name="${lat_label}_rocker_joint" type="continuous">
             <origin rpy="0 0 0" xyz="0.071 ${reflect * 0.155} 0.0118"/>
@@ -55,14 +60,10 @@
             <limit
                 lower="${-math_pi_over_4}"
-                upper="${math_pi_over_4}"
-                effort="100.0"
-                velocity="30.0" />
-            <parent link="${parent}" />
-            <child link="${lat_label}_rocker_link" />
+            upper="${math_pi_over_4}"
+            effort="100.0"
+            velocity="30.0" />
+        <parent link="${parent}" />
+        <child link="${lat_label}_rocker_link" />
         </joint>
-        <gazebo reference="${lat_label}_rocker_joint">
-            <provideFeedback>true</provideFeedback>
-            <implicitSpringDamper>true</implicitSpringDamper>
-        </gazebo>
     </xacro:macro>
 </robot>

File: rover_description/urdf/bases/turnbuckle.urdf.xacro (robot description, xacro)
@@ -27,5 +27,6 @@
                     <geometry>
                         <mesh>
-                            <uri>package://rover_description/meshes/bases/turnbuckle.stl</uri>
+                            <!-- <uri>package://rover_description/meshes/bases/turnbuckle.stl</uri> -->
+                            <uri>file://$(find rover_description)/meshes/bases/turnbuckle.stl</uri>
                         </mesh>
                         <!-- <cylinder>
@@ -34,9 +35,4 @@
                         </cylinder> -->
                     </geometry>
-                    <material>
-                        <script>
-                            <name>Gazebo/Blue</name>
-                        </script>
-                    </material>
                 </visual>
                 <collision name="${lat_label}_turnbuckle_collision">
@@ -61,9 +57,10 @@
                 </inertial>
             </link>
-            <joint name="back_${lat_label}_turnbuckle_joint" type="ball">
-                <pose>-0.035 0 0 0 0 0</pose>
+            <joint name="back_${lat_label}_turnbuckle_joint" type="fixed">
+                <pose>-0.035 0 1.0 0 0 0</pose>
                 <parent>diff_brace_link</parent>
                 <child>${lat_label}_turnbuckle_link</child>
             </joint>
+<!--
             <joint name="front_${lat_label}_turnbuckle_joint" type="ball">
                 <pose>0.035 0 0 0 0 0</pose>
@@ -71,4 +68,5 @@
                 <child>${lat_label}_turnbuckle_link</child>
             </joint>
+-->
         </gazebo>
     </xacro:macro>

File: rover_description/urdf/sensors/all_sensors.urdf.xacro (robot description, xacro)
@@ -22,5 +22,5 @@
   <!-- Hokuyo -->
   <xacro:include filename="$(find rover_description)/urdf/sensors/hokuyo.urdf.xacro" />
-  <!-- Hokuyo -->
+  <!-- XTion -->
   <xacro:include filename="$(find rover_description)/urdf/sensors/asus_xtion.urdf.xacro" />
 </robot>

File: rover_description/urdf/sensors/asus_xtion.urdf.xacro (robot description, xacro)
@@ -18,13 +18,13 @@
 # SOFTWARE. -->
 <robot name="sensor_asus_xtion" xmlns:xacro="http://www.ros.org/wiki/xacro">
-  <xacro:macro name="sensor_asus_xtion" params="prefix parent *origin ">
-    <xacro:property name="math_pi_over_2" value="1.5707963267948966" />
-    <joint name="${prefix}_joint" type="fixed">
+  <xacro:macro name="sensor_asus_xtion" params="prefix parent *origin">
+   <xacro:property name="math_pi_over_2" value="1.5707963267948966" />
+   <joint name="${prefix}_joint" type="fixed">
         <axis xyz="1 0 0"/>
-        <xacro:insert_block name="origin"/>
+        <xacro:insert_block name="origin" />
         <parent link="${parent}"/>
         <child link="${prefix}_link"/>
-    </joint>
-    <link name="${prefix}_link">
+   </joint>
+   <link name="${prefix}_link">
       <visual>
         <origin rpy="${math_pi_over_2} 0 ${math_pi_over_2}" xyz="0 0 0"/>
@@ -47,10 +47,10 @@
       </inertial>
     </link>
-    <joint name="camera_frame_joint" type="fixed">
+   <joint name="camera_frame_joint" type="fixed">
       <origin xyz="0 0 0" rpy="-${math_pi_over_2} 0 -${math_pi_over_2}" />
       <parent link="${prefix}_link" />
       <child link="camera_frame" />
-    </joint>
-    <link name="camera_frame">
+   </joint>
+   <link name="camera_frame">
       <inertial>
         <mass value="0.001" />
@@ -60,9 +60,14 @@
           izz="0.001" />
       </inertial>
-    </link>
-    <gazebo reference="${prefix}_link">
-      <sensor name="camera" type="depth">
+   </link>
+   <gazebo reference="${prefix}_link">
+      <plugin filename="libignition-gazebo-sensors-system.so"
+              name="ignition::gazebo::systems::Sensors">
+        <render_engine>ogre2</render_engine>
+      </plugin>
+      <sensor name="camera" type="depth_camera">
+        <update_rate>30</update_rate>
+        <topic> depth_camera</topic>
         <visualize>true</visualize>
-        <update_rate>30</update_rate>
         <camera>
           <horizontal_fov>${63.0*2*math_pi_over_2/180.0}</horizontal_fov>
@@ -84,69 +89,23 @@
           </distortion>
         </camera>
-        <plugin name="depth_camera_controller" filename="libgazebo_ros_camera.so">
-          <ros>
-            <qos>
-              <topic name="/camera/camera_info">
-                <publisher>
-                  <reliability>best_effort</reliability>
-                </publisher>
-              </topic>
-              <topic name="/camera/image_raw">
-                <publisher>
-                  <reliability>best_effort</reliability>
-                </publisher>
-              </topic>
-              <topic name="/camera/image_raw/compressed">
-                <publisher>
-                  <reliability>best_effort</reliability>
-                </publisher>
-              </topic>
-              <topic name="/camera/image_raw/compressedDepth">
-                <publisher>
-                  <reliability>best_effort</reliability>
-                </publisher>
-              </topic>
-              <topic name="/camera/image_raw/theora">
-                <publisher>
-                  <reliability>best_effort</reliability>
-                </publisher>
-              </topic>
-              <topic name="/camera/points">
-                <publisher>
-                  <reliability>best_effort</reliability>
-                </publisher>
-              </topic>
-              <topic name="/camera/depth/camera_info">
-                <publisher>
-                  <reliability>best_effort</reliability>
-                </publisher>
-              </topic>
-              <topic name="/camera/depth/image_raw">
-                <publisher>
-                  <reliability>best_effort</reliability>
-                </publisher>
-              </topic>
-              <topic name="/camera/depth/image_raw/compressed">
-                <publisher>
-                  <reliability>best_effort</reliability>
-                </publisher>
-              </topic>
-              <topic name="/camera/depth/image_raw/compressedDepth">
-                <publisher>
-                  <reliability>best_effort</reliability>
-                </publisher>
-              </topic>
-             <topic name="/camera/depth/image_raw/theora">
-                <publisher>
-                  <reliability>best_effort</reliability>
-                </publisher>
-              </topic>
-            </qos>
-          </ros>
-          <frame_name>camera_frame</frame_name>
-          <min_depth>0.3</min_depth>
-          <max_depth>8.0</max_depth>
-        </plugin>
       </sensor>
+<!-- CAMERA CODE THROWING GAZEBO ERROR.... kmn 6/29
+        <plugin filename="ImageDisplay" name="front_depth_camera">
+              <topic name="/camera/depth_image">
+              <ignition-gui>
+                <title>front depth camera</title>
+                <property key="state" type="string">floating</property>
+                <property type="double" key="height">300</property>
+                <property type="double" key="width">300</property>
+                <property type="double" key="x">1</property>
+                <property type="double" key="y">1</property>
+                <property type="double" key="z">1</property>
+              </ignition-gui>
+            <frame_name>camera_frame</frame_name>
+            <min_depth>0.3</min_depth>
+            <max_depth>8.0</max_depth>
+          </plugin>
+      </sensor>
+-->
     </gazebo>
   </xacro:macro>

File: rover_description/urdf/sensors/hokuyo.urdf.xacro (robot description, xacro)
@@ -43,7 +43,4 @@
       </inertial>
     </link>
-    <gazebo reference="${prefix}_base_link">
-        <material>Gazebo/DarkGrey</material>
-    </gazebo>
     <link name="${prefix}_link">
     </link>
@@ -54,43 +51,34 @@
     </joint>
     <gazebo reference="${prefix}_link">
-            <sensor type="gpu_ray" name="hokuyo_sensor">
-                <pose>0 0 0 0 0 0</pose>
-                <visualize>true</visualize>
-                <update_rate>50</update_rate>
-                <ray>
-                    <scan>
-                        <horizontal>
-                            <samples>30</samples>
-                            <resolution>1</resolution>
-                            <min_angle>${min_angle}</min_angle>
-                            <max_angle>${max_angle}</max_angle>
-                        </horizontal>
-                    </scan>
-                    <range>
-                        <min>0.06</min>
-                        <max>5.0</max>
-                        <resolution>0.004359297</resolution>
-                    </range>
-                    <noise>
-                        <type>gaussian</type>
-                        <mean>0.0</mean>
-                        <stddev>0.01</stddev>
-                    </noise>
-                </ray>
-                <plugin name="${prefix}_controller" filename="libgazebo_ros_ray_sensor.so">
-                  <ros>
-                    <remapping>~/out:=scan</remapping>
-                    <qos>
-                      <topic name="scan">
-                        <publisher>
-                          <reliability>best_effort</reliability>
-                        </publisher>
-                      </topic>
-                    </qos>
-                  </ros>
-                  <output_type>sensor_msgs/LaserScan</output_type>
-                  <frame_name>${prefix}_link</frame_name>
-                </plugin>
-            </sensor>
+      <plugin filename="libignition-gazebo-sensors-system.so"
+              name="ignition::gazebo::systems::Sensors">
+        <render_engine>ogre2</render_engine>
+      </plugin>
+      <sensor type="gpu_lidar" name="hokuyo_sensor">
+          <pose>0 0 0 0 0 0</pose>
+          <visualize>true</visualize>
+          <update_rate>50</update_rate>
+          <topic>sensor_msgs/LaserScan</topic>
+          <ray>
+              <scan>
+                  <horizontal>
+                      <samples>30</samples>
+                      <resolution>1</resolution>
+                      <min_angle>${min_angle}</min_angle>
+                      <max_angle>${max_angle}</max_angle>
+                  </horizontal>
+              </scan>
+              <range>
+                  <min>0.06</min>
+                  <max>5.0</max>
+                  <resolution>0.004359297</resolution>
+              </range>
+              <noise>
+                  <type>gaussian</type>
+                  <mean>0.0</mean>
+                  <stddev>0.01</stddev>
+              </noise>
+          </ray>
+      </sensor>
     </gazebo>
   </xacro:macro>

File: rover_description/urdf/sensors/imu.urdf.xacro (robot description, xacro)
@@ -19,10 +19,4 @@
 <robot name="sensor_imu" xmlns:xacro="http://www.ros.org/wiki/xacro">
   <xacro:macro name="sensor_imu" params="prefix parent *origin">
-    <joint name="${prefix}_joint" type="fixed">
-        <axis xyz="1 0 0"/>
-        <xacro:insert_block name="origin"/>
-        <parent link="${parent}"/>
-        <child link="${prefix}_link"/>
-    </joint>
     <link name="${prefix}_link">
       <inertial>
@@ -45,80 +39,18 @@
       </collision>
     </link>
+    <joint name="${prefix}_joint" type="fixed">
+        <axis xyz="1 0 0"/>
+        <xacro:insert_block name="origin"/>
+        <parent link="${parent}"/>
+        <child link="${prefix}_link"/>
+    </joint>
     <gazebo reference="${prefix}_link">
-        <material>Gazebo/Blue</material>
-    </gazebo>
-    <gazebo reference="${prefix}_link">
+      <plugin filename="libignition-gazebo-imu-system.so"
+        name="ignition::gazebo::systems::Sensors">
+      </plugin>
       <sensor name="imu_sensor" type="imu">
-        <plugin filename="libgazebo_ros_imu_sensor.so" name="imu_controller">
-          <ros>
-            <remapping>~/out:=imu</remapping>
-            <qos>
-              <topic name="imu">
-                <publisher>
-                  <reliability>best_effort</reliability>
-                </publisher>
-              </topic>
-            </qos>
-          </ros>
-          <initial_orientation_as_reference>false</initial_orientation_as_reference>
-          <frame_name>${prefix}_link</frame_name>
-        </plugin>
-        <always_on>true</always_on>
-        <update_rate>200</update_rate>
-        <visualize>true</visualize>
-        <imu>
-          <angular_velocity>
-            <x>
-              <noise type="gaussian">
-                <mean>0.0</mean>
-                <stddev>2e-4</stddev>
-                <bias_mean>0.0000075</bias_mean>
-                <bias_stddev>0.0000008</bias_stddev>
-              </noise>
-            </x>
-            <y>
-              <noise type="gaussian">
-                <mean>0.0</mean>
-                <stddev>2e-4</stddev>
-                <bias_mean>0.0000075</bias_mean>
-                <bias_stddev>0.0000008</bias_stddev>
-              </noise>
-            </y>
-            <z>
-              <noise type="gaussian">
-                <mean>0.0</mean>
-                <stddev>2e-4</stddev>
-                <bias_mean>0.0000075</bias_mean>
-                <bias_stddev>0.0000008</bias_stddev>
-              </noise>
-            </z>
-          </angular_velocity>
-          <linear_acceleration>
-            <x>
-              <noise type="gaussian">
-                <mean>0.0</mean>
-                <stddev>1.7e-2</stddev>
-                <bias_mean>0.1</bias_mean>
-                <bias_stddev>0.001</bias_stddev>
-              </noise>
-            </x>
-            <y>
-              <noise type="gaussian">
-                <mean>0.0</mean>
-                <stddev>1.7e-2</stddev>
-                <bias_mean>0.1</bias_mean>
-                <bias_stddev>0.001</bias_stddev>
-              </noise>
-            </y>
-            <z>
-              <noise type="gaussian">
-                <mean>0.0</mean>
-                <stddev>1.7e-2</stddev>
-                <bias_mean>0.1</bias_mean>
-                <bias_stddev>0.001</bias_stddev>
-              </noise>
-            </z>
-          </linear_acceleration>
-        </imu>
+            <always_on>true</always_on>
+            <update_rate>200</update_rate>
+            <visualize>true</visualize>
       </sensor>
     </gazebo>

File: rover_description/urdf/wheels/corner.urdf.xacro (robot description, xacro)
@@ -46,7 +46,4 @@
                 x="${corner_box_length}" y="${corner_box_width}" z="${corner_box_depth}" />
         </link>
-        <gazebo reference="${lon_label}_${lat_label}_corner_link">
-            <material>Gazebo/White</material>
-        </gazebo>
     </xacro:macro>
     <!-- front joint -->
@@ -60,7 +57,4 @@
             <dynamics damping="0.0" friction="0.0"/>
         </joint>
-        <gazebo reference="front_${lat_label}_corner_joint">
-            <provideFeedback>true</provideFeedback>
-        </gazebo>
     </xacro:macro>
     <!-- back joint -->
@@ -74,7 +68,4 @@
             <dynamics damping="0.0" friction="0.0"/>
         </joint>
-        <gazebo reference="back_${lat_label}_corner_joint">
-            <provideFeedback>true</provideFeedback>
-        </gazebo>
     </xacro:macro>
 </robot>
