Commit message: all three sensors not crashing

File: rover_description/urdf/wheels/wheel.urdf.xacro (robot description, xacro)
@@ -45,5 +45,4 @@
         </link>
         <gazebo reference="${lon_label}_${lat_label}_wheel_link">
-            <material>Gazebo/DarkGray</material>
 			<mu1 value="100.0"/>
 			<mu2 value="100.0"/>
@@ -64,7 +63,4 @@
             <dynamics damping="0.0" friction="0.0"/>
         </joint>
-        <gazebo reference="${lon_label}_${lat_label}_wheel_joint">
-            <provideFeedback>true</provideFeedback>
-        </gazebo>
     </xacro:macro>
     <!-- mid wheel joint -->
@@ -78,7 +74,4 @@
             <dynamics damping="0.0" friction="0.0"/>
         </joint>
-        <gazebo reference="mid_${lat_label}_wheel_joint">
-            <provideFeedback>true</provideFeedback>
-        </gazebo>
     </xacro:macro>
 </robot>
